Commit message: add the vacuum gripper and another realsense mounting on a gripper

File: src/mobile_robot/urdf/manipulator.xacro (robot description, xacro)
@@ -1,22 +1,15 @@
 <?xml version="1.0"?>
-<robot name="mobile_manipulator" xmlns:xacro="http://www.ros.org/wiki/xacro">
-  <xacro:include filename="$(find-pkg-share ur_description)/urdf/ur5.urdf.xacro"/>
-  <link name="ur5_mount_link">
-    <visual>
-      <geometry>
-        <cylinder radius="0.12" length="0.05"/>
-      </geometry>
-    </visual>
-  </link>
-  <joint name="base_to_mount" type="fixed">
-    <parent link="base_link"/>
-    <child link="ur5_mount_link"/>
-    <origin xyz="0 0 0.4" rpy="0 0 0"/>
-  </joint>
-  <xacro:ur5_robot prefix="ur5_"/>
-  <joint name="mount_to_ur5" type="fixed">
-    <parent link="ur5_mount_link"/>
-    <child link="ur5_base_link"/>
-    <origin xyz="0 0 0" rpy="0 0 0"/>
-  </joint>
+<robot xmlns:xacro="http://www.ros.org/wiki/xacro">
+  <xacro:include filename="$(find ur_description)/urdf/ur_macro.xacro"/>
+  <xacro:ur_robot
+    name="ur5"
+    tf_prefix="ur5_"
+    parent="base_link"
+    joint_limits_parameters_file="$(find ur_description)/config/ur5/joint_limits.yaml"
+    kinematics_parameters_file="$(find ur_description)/config/ur5/default_kinematics.yaml"
+    physical_parameters_file="$(find ur_description)/config/ur5/physical_parameters.yaml"
+    visual_parameters_file="$(find ur_description)/config/ur5/visual_parameters.yaml">
+    <origin xyz="0.35 0.0 0.20" rpy="0 0 0" />
+    <xacro:property name="initial_positions" value="${dict(shoulder_pan_joint=1.57, shoulder_lift_joint=-1.57, elbow_joint=0.0, wrist_1_joint=-1.57, wrist_2_joint=0.0, wrist_3_joint=0.0)}" />
+  </xacro:ur_robot>
 </robot>

File: src/mobile_robot/urdf/robot.urdf.xacro (robot description, xacro)
@@ -1,18 +1,15 @@
 <?xml version="1.0"?>
 <robot xmlns:xacro="http://www.ros.org/wiki/xacro" name="mobile_robot">
+  <xacro:include filename="realsense_sensor.xacro"/>
   <xacro:include filename="robot.xacro"/>
   <xacro:include filename="ros2_control.xacro"/>
-  <xacro:include filename="$(find ur_description)/urdf/ur_macro.xacro"/>
-  <xacro:include filename="Realsense.xacro"/>
-  <xacro:ur_robot
-    name="ur5"
-    tf_prefix="ur5_"
-    parent="base_link"
-    joint_limits_parameters_file="$(find ur_description)/config/ur5/joint_limits.yaml"
-    kinematics_parameters_file="$(find ur_description)/config/ur5/default_kinematics.yaml"
-    physical_parameters_file="$(find ur_description)/config/ur5/physical_parameters.yaml"
-    visual_parameters_file="$(find ur_description)/config/ur5/visual_parameters.yaml">
-    <origin xyz="0.35 0.0 0.20" rpy="0 0 0" />
-    <xacro:property name="initial_positions" value="${dict(shoulder_pan_joint=1.57, shoulder_lift_joint=-1.57, elbow_joint=0.0, wrist_1_joint=-1.57, wrist_2_joint=0.0, wrist_3_joint=0.0)}" />
-  </xacro:ur_robot>
+  <xacro:include filename="manipulator.xacro"/>
+  <xacro:include filename="vacuum_gripper.xacro"/>
+  <gazebo>
+    <plugin
+      filename="gz-sim-sensors-system"
+      name="gz::sim::systems::Sensors">
+      <render_engine>ogre2</render_engine>
+    </plugin>
+  </gazebo>
 </robot>

File: src/mobile_robot/urdf/robot.xacro (robot description, xacro)
@@ -110,5 +110,5 @@
   </link>
   <joint name="camera_joint" type="fixed">
-    <origin xyz="0.474 0.0 0.1355" rpy="0 0 0"/>
+    <origin xyz="0.474 0.0 0.1355" rpy="-3.141592653589793 -1.5707963267948966 0"/>
     <parent link="base_link"/><child link="realsense"/>
   </joint>
@@ -151,3 +151,6 @@
     <kd>10.0</kd>
   </gazebo>
+  <xacro:realsense_sensor name="base_camera" topics_ns="base_cam" parent_link="realsense">
+    <origin xyz="0.0 0 0.0" rpy="0 0 0"/>
+  </xacro:realsense_sensor>
 </robot>
