Commit message: finally we have 2Dlidar inside our robot

File: src/mobile_robot/urdf/robot.urdf.xacro (robot description, xacro)
@@ -6,3 +6,5 @@
   <xacro:include filename="robot.xacro"/>
   <xacro:include filename="ros2_control.xacro"/>
+  <xacro:include filename="inertial_macros.xacro"/>
+  <xacro:include filename="lidar.xacro"/>
 </robot>

File: src/mobile_robot/urdf/robot.xacro (robot description, xacro)
@@ -1,4 +1,10 @@
 <?xml version="1.0"?>
 <robot name="mobile_robot" xmlns:xacro="http://www.ros.org/wiki/xacro">
+  <material name="red">
+        <color rgba="1 0 0 1"/>
+  </material>
+  <material name="black">
+        <color rgba="0 0 0 1"/>
+    </material>
   <link name="base_link"/>
   <link name="mobile_base">

Commit message: change it to 4 wheels but not add manipulator yet

File: src/mobile_robot/urdf/robot.urdf.xacro (robot description, xacro)
@@ -1,10 +1,7 @@
 <?xml version="1.0"?>
 <robot xmlns:xacro="http://www.ros.org/wiki/xacro" name="mobile_robot">
-  <!-- parameter define  -->
-  <xacro:arg name="controller_yaml" default=""/>
   <!-- shitty file for our robot -->
   <xacro:include filename="robot.xacro"/>
   <xacro:include filename="ros2_control.xacro"/>
-  <xacro:include filename="inertial_macros.xacro"/>
-  <xacro:include filename="lidar.xacro"/>
+  <!-- <xacro:include filename="lidar.xacro"/> -->
 </robot>

File: src/mobile_robot/urdf/robot.xacro (robot description, xacro)
@@ -1,113 +1,209 @@
-<?xml version="1.0"?>
-<robot name="mobile_robot" xmlns:xacro="http://www.ros.org/wiki/xacro">
-  <material name="red">
-        <color rgba="1 0 0 1"/>
-  </material>
-  <material name="black">
-        <color rgba="0 0 0 1"/>
-    </material>
-  <link name="base_link"/>
-  <link name="mobile_base">
-    <inertial>
-      <origin xyz="-8.80e-06 -5.08e-06 0.025" rpy="0 0 0" />
-      <mass value="3"/>
-      <inertia ixx="0.31" iyy="0.31" izz="0.59" ixy="0" iyz="0" ixz="0" />
-    </inertial>
-    <visual>
-      <origin xyz="0 0 0" rpy="0 0 0" />
-      <geometry>
-        <mesh filename="package://mobile_robot/meshes/mobile_base.stl" scale="0.001 0.001 0.001" />
-      </geometry>
-    </visual>
-    <collision>
-      <origin xyz="0 0 0.025" rpy="0 0 0" />
-      <geometry>
-        <cylinder radius="0.13" length="0.05"/>
-      </geometry>
-    </collision>
-  </link>
-  <joint name="base_link_to_mobile_base" type="fixed">
-    <parent link="base_link"/>
-    <child link="mobile_base"/>
-    <origin xyz="0 0 0.035" rpy="0 0 0"/>
-  </joint>
-  <xacro:macro name="omni_wheel" params="prefix joint_name joint_xyz joint_rpy v_xyz v_rpy mesh_num">
-    <link name="Omni_wheel_single_part_${prefix}">
-      <inertial>
-        <origin xyz="0 0 0" rpy="0 0 0" />
-        <mass value="1" />
-        <inertia ixx="0.023" iyy="0.023" izz="0.041" ixy="0" iyz="0" ixz="0" />
-      </inertial>
-      <visual>
-        <origin xyz="${v_xyz}" rpy="${v_rpy}" />
-        <geometry>
-          <mesh filename="package://mobile_robot/meshes/Omni_wheel_single_part_${mesh_num}.stl" scale="0.001 0.001 0.001" />
-        </geometry>
-      </visual>
-      <collision>
-        <origin xyz="0 0 0" rpy="0 0 0" />
-        <geometry><cylinder radius="0.06" length="0.03"/></geometry>
-      </collision>
-    </link>
-    <joint name="${joint_name}" type="continuous">
-      <origin xyz="${joint_xyz}" rpy="${joint_rpy}"/>
-      <parent link="mobile_base"/>
-      <child link="Omni_wheel_single_part_${prefix}"/>
-      <axis xyz="0 0 1"/>
-      <dynamics damping="0.0" friction="0.0"/>
-    </joint>
-    <gazebo reference="Omni_wheel_single_part_${prefix}">
-      <mu1 value="2.0"/>
-      <mu2 value="0.01"/>
-      <fdir1 value="1 0 0"/>
-      <kp value="10000000.0"/>
-      <kd value="1.0"/>
-      <minDepth value="0.001"/>
-      <maxVel value="0.1"/>
-    </gazebo>
-  </xacro:macro>
-  <xacro:omni_wheel
-    prefix="1"
-    mesh_num="2"
-    joint_name="mobile_base_Revolute_1"
-    joint_xyz="0.0 0.1766 0.025"
-    joint_rpy="-1.5708 0 0"
-    v_xyz="2.22e-08 0.018 0.715"
-    v_rpy="1.5708 -1.5708 0"/>
-  <xacro:omni_wheel
-    prefix="2"
-    mesh_num="3"
-    joint_name="mobile_base_Revolute_2"
-    joint_xyz="0.15294 -0.0883 0.025"
-    joint_rpy="-1.5708 0 -2.0944"
-    v_xyz="2.55e-08 0.018 0.715"
-    v_rpy="1.5708 -1.5708 0"/>
-  <xacro:omni_wheel
-    prefix="3"
-    mesh_num="1"
-    joint_name="mobile_base_Revolute_3"
-    joint_xyz="-0.15294 -0.0883 0.025"
-    joint_rpy="-1.5708 0 2.0944"
-    v_xyz="-2.52e-08 0.018 -0.738"
-    v_rpy="1.5708 1.5708 0"/>
-  <physics type="ode">
-    <real_time_update_rate>1000</real_time_update_rate>
-    <max_step_size>0.001</max_step_size>
-  </physics>
-  <gazebo reference="ground_plane">
-    <mu1>100.0</mu1>
-    <mu2>100.0</mu2>
-  </gazebo>
+<?xml version="1.0" encoding="utf-8"?>
+<robot name="4_wheel_mobile_assem">
+  <!-- DUMMY ROOT TO SATISFY KDL -->
+  <link name="base_footprint"/>
+  <joint name="base_joint" type="fixed">
+    <parent link="base_footprint"/>
+    <child link="base_link"/>
+  </joint>
+  <!-- BASE LINK -->
+  <link name="base_link">
+    <inertial>
+      <origin xyz="0.00628429000821322 0.0 0.09385603458840618" rpy="0.0 0.0 0.0"/>
+      <mass value="987.3844207986756"/>
+      <inertia ixx="40.57825725748298" iyy="87.33699297862528" izz="122.02543924646025"
+               ixy="0.0" iyz="0.0" ixz="-0.6159379832813523"/>
+    </inertial>
+    <visual name="base_link_visual">
+      <origin xyz="0.0 0.0 0.0" rpy="0.0 0.0 0.0"/>
+      <geometry>
+        <mesh filename="package://mobile_robot/meshes/base_link.stl" scale="0.001 0.001 0.001"/>
+      </geometry>
+    </visual>
+    <collision name="base_link_collision">
+      <origin xyz="0.0 0.0 0.0" rpy="0.0 0.0 0.0"/>
+      <geometry>
+        <mesh filename="package://mobile_robot/meshes/base_link.stl" scale="0.001 0.001 0.001"/>
+      </geometry>
+    </collision>
+  </link>
+  <!-- WHEEL 1 (Front Left) -->
+  <link name="omni_wheel_1">
+    <inertial>
+      <origin xyz="-7.970962720094121e-06 -6.877816728989572e-06 -0.01147703773614026" rpy="0.0 0.0 0.0"/>
+      <mass value="1.7319883752876981"/>
+      <inertia ixx="0.002224867748533532" iyy="0.0022250042535725822" izz="0.004048574614964773"
+               ixy="-4.500394812853581e-07" iyz="4.899447401951473e-08" ixz="5.879718084633723e-08"/>
+    </inertial>
+    <visual name="omni_wheel_1_visual">
+      <origin xyz="2.2665481083095073e-08 0.018031436920169994 0.7154857177799999" rpy="1.5707963267948968 -1.5707963267948966 0"/>
+      <geometry>
+        <mesh filename="package://mobile_robot/meshes/Omni_wheel.stl" scale="0.001 0.001 0.001"/>
+      </geometry>
+    </visual>
+    <collision name="omni_wheel_1_collision">
+      <origin xyz="2.2665481083095073e-08 0.018031436920169994 0.7154857177799999" rpy="1.5707963267948968 -1.5707963267948966 0"/>
+      <geometry>
+        <mesh filename="package://mobile_robot/meshes/Omni_wheel.stl" scale="0.001 0.001 0.001"/>
+      </geometry>
+    </collision>
+  </link>
+  <joint name="wheel_1_joint" type="continuous">
+    <origin xyz="-0.375 0.395 0.025" rpy="-1.5707963267948966 0.0 0.0"/>
+    <parent link="base_link"/>
+    <child link="omni_wheel_1"/>
+    <axis xyz="0.0 0.0 1.0"/>
+    <dynamics damping="0.1" friction="0.1"/>
+  </joint>
+  <!-- WHEEL 2 (Front Right) -->
+  <link name="omni_wheel_2">
+    <inertial>
+      <origin xyz="-7.970962720094121e-06 -6.877816728980691e-06 -0.01147703773614026" rpy="0.0 0.0 0.0"/>
+      <mass value="1.7319883752876981"/>
+      <inertia ixx="0.002224867748534254" iyy="0.002225004253573304" izz="0.004048574614964745"
+               ixy="-4.5003948128188864e-07" iyz="4.8994474016045286e-08" ixz="5.8797180790826076e-08"/>
+    </inertial>
+    <visual name="omni_wheel_2_visual">
+      <origin xyz="2.2665481083095073e-08 0.018031436920170004 0.7154857177799999" rpy="1.5707963267948968 -1.5707963267948966 0"/>
+      <geometry>
+        <mesh filename="package://mobile_robot/meshes/Omni_wheel.stl" scale="0.001 0.001 0.001"/>
+      </geometry>
+    </visual>
+    <collision name="omni_wheel_2_collision">
+      <origin xyz="2.2665481083095073e-08 0.018031436920170004 0.7154857177799999" rpy="1.5707963267948968 -1.5707963267948966 0"/>
+      <geometry>
+        <mesh filename="package://mobile_robot/meshes/Omni_wheel.stl" scale="0.001 0.001 0.001"/>
+      </geometry>
+    </collision>
+  </link>
+  <joint name="wheel_2_joint" type="continuous">
+    <origin xyz="0.375 0.395 0.025" rpy="-1.5707963267948966 0.0 0.0"/>
+    <parent link="base_link"/>
+    <child link="omni_wheel_2"/>
+    <axis xyz="0.0 0.0 1.0"/>
+    <dynamics damping="0.1" friction="0.1"/>
+  </joint>
+  <!-- WHEEL 3 (Rear Left) -->
+  <link name="omni_wheel_3">
+    <inertial>
+      <origin xyz="-7.970962720094121e-06 6.877816728985131e-06 -0.011522962255859852" rpy="0.0 0.0 0.0"/>
+      <mass value="1.7319883752876981"/>
+      <inertia ixx="0.0022248677485343094" iyy="0.0022250042535733594" izz="0.004048574614964773"
+               ixy="4.5003948128188864e-07" iyz="4.8994474016045286e-08" ixz="-5.8797180790826076e-08"/>
+    </inertial>
+    <visual name="omni_wheel_3_visual">
+      <origin xyz="2.2665481083095073e-08 -0.01803143692017 -0.7384857177720001" rpy="-1.5707963267948966 1.5707963267948966 0"/>
+      <geometry>
+        <mesh filename="package://mobile_robot/meshes/Omni_wheel.stl" scale="0.001 0.001 0.001"/>
+      </geometry>
+    </visual>
+    <collision name="omni_wheel_3_collision">
+      <origin xyz="2.2665481083095073e-08 -0.01803143692017 -0.7384857177720001" rpy="-1.5707963267948966 1.5707963267948966 0"/>
+      <geometry>
+        <mesh filename="package://mobile_robot/meshes/Omni_wheel.stl" scale="0.001 0.001 0.001"/>
+      </geometry>
+    </collision>
+  </link>
+  <joint name="wheel_3_joint" type="continuous">
+    <origin xyz="-0.375 -0.395 0.025" rpy="1.5707963267948966 0.0 0.0"/>
+    <parent link="base_link"/>
+    <child link="omni_wheel_3"/>
+    <axis xyz="0.0 0.0 1.0"/>
+    <dynamics damping="0.1" friction="0.1"/>
+  </joint>
+  <!-- WHEEL 4 (Rear Right) -->
+  <link name="omni_wheel_4">
+    <inertial>
+      <origin xyz="-7.970962720094121e-06 6.877816728985131e-06 -0.011522962255859852" rpy="0.0 0.0 0.0"/>
+      <mass value="1.7319883752876981"/>
+      <inertia ixx="0.0022248677485343094" iyy="0.002225004253573415" izz="0.004048574614964745"
+               ixy="4.500394812853581e-07" iyz="4.8994474016045286e-08" ixz="-5.879718081858165e-08"/>
+    </inertial>
+    <visual name="omni_wheel_4_visual">
+      <origin xyz="2.2665481083095073e-08 -0.01803143692017 -0.7384857177720001" rpy="-1.5707963267948966 1.5707963267948966 0"/>
+      <geometry>
+        <mesh filename="package://mobile_robot/meshes/Omni_wheel.stl" scale="0.001 0.001 0.001"/>
+      </geometry>
+    </visual>
+    <collision name="omni_wheel_4_collision">
+      <origin xyz="2.2665481083095073e-08 -0.01803143692017 -0.7384857177720001" rpy="-1.5707963267948966 1.5707963267948966 0"/>
+      <geometry>
+        <mesh filename="package://mobile_robot/meshes/Omni_wheel.stl" scale="0.001 0.001 0.001"/>
+      </geometry>
+    </collision>
+  </link>
+  <joint name="wheel_4_joint" type="continuous">
+    <origin xyz="0.375 -0.395 0.025" rpy="1.5707963267948966 0.0 0.0"/>
+    <parent link="base_link"/>
+    <child link="omni_wheel_4"/>
+    <axis xyz="0.0 0.0 1.0"/>
+    <dynamics damping="0.1" friction="0.1"/>
+  </joint>
+  <!-- CAMERA (RealSense D455) -->
+  <link name="realsense">
+    <inertial>
+      <origin xyz="6.359106729602714e-05 -0.0001583183035289228 0.013103406900131134" rpy="0.0 0.0 0.0"/>
+      <mass value="0.4224343307990776"/>
+      <inertia ixx="0.0005263815553470524" iyy="4.808114888894821e-05" izz="0.0005349726197919043"
+               ixy="-3.4306312466689594e-07" iyz="3.9088259249671483e-07" ixz="2.188450578845258e-07"/>
+    </inertial>
+    <visual name="realsense_visual">
+      <origin xyz="-4.5257177916369075e-09 1.5070762415803906e-11 0.025999999999999943" rpy="0.0 0.0 -1.5707963267948968"/>
+      <geometry>
+        <mesh filename="package://mobile_robot/meshes/Realsense_D455.stl" scale="0.001 0.001 0.001"/>
+      </geometry>
+    </visual>
+    <collision name="realsense_collision">
+      <origin xyz="-4.5257177916369075e-09 1.5070762415803906e-11 0.025999999999999943" rpy="0.0 0.0 -1.5707963267948968"/>
+      <geometry>
+        <mesh filename="package://mobile_robot/meshes/Realsense_D455.stl" scale="0.001 0.001 0.001"/>
+      </geometry>
+    </collision>
+  </link>
+  <joint name="camera_joint" type="fixed">
+    <origin xyz="0.474 0.0 0.1355" rpy="-3.141592653589793 -1.5707963267948966 0"/>
+    <parent link="base_link"/>
+    <child link="realsense"/>
+  </joint>
+  <!-- GAZEBO SPECIFIC SETTINGS -->
+  <!-- Global Physics -->
   <gazebo>
-    <plugin name="gazebo_ros_p3d" filename="libgazebo_ros_p3d.so">
-      <ros>
-        <namespace>/ground_truth</namespace>
-      </ros>
-      <body_name>base_link</body_name>
-      <frame_name>world</frame_name>
-      <update_rate>50.0</update_rate>
-      <xyz_offset>0 0 0</xyz_offset>
-      <rpy_offset>0 0 0</rpy_offset>
-      <gaussian_noise>0.0</gaussian_noise>
+    <physics type="ode">
+      <real_time_update_rate>1000</real_time_update_rate>
+      <max_step_size>0.001</max_step_size>
+    </physics>
+  </gazebo>
+  <!-- Material colors for Gazebo -->
+  <gazebo reference="base_link">
+    <material>Gazebo/Grey</material>
+  </gazebo>
+  <gazebo reference="omni_wheel_1">
+    <material>Gazebo/Black</material>
+    <mu1>0.8</mu1>
+    <mu2>0.8</mu2>
+  </gazebo>
+  <gazebo reference="omni_wheel_2">
+    <material>Gazebo/Black</material>
+    <mu1>0.8</mu1>
+    <mu2>0.8</mu2>
+  </gazebo>
+  <gazebo reference="omni_wheel_3">
+    <material>Gazebo/Black</material>
+    <mu1>0.8</mu1>
+    <mu2>0.8</mu2>
+  </gazebo>
+  <gazebo reference="omni_wheel_4">
+    <material>Gazebo/Black</material>
+    <mu1>0.8</mu1>
+    <mu2>0.8</mu2>
+  </gazebo>
+  <gazebo reference="realsense">
+    <material>Gazebo/DarkGrey</material>
+  </gazebo>
+  <gazebo>
+    <plugin name="gazebo_ros_state" filename="libgazebo_ros_state.so">
+        <ros>
+        <namespace>/</namespace>
+        </ros>
     </plugin>
   </gazebo>

File: src/mobile_robot/urdf/ros2_control.xacro (robot description, xacro)
@@ -9,6 +9,6 @@
     <joint name="mobile_base_Revolute_1">
       <command_interface name="effort">
-        <param name="min">-5</param>
-        <param name="max">5</param>
+        <param name="min">-10</param>
+        <param name="max">10</param>
       </command_interface>
       <state_interface name="position"/>
@@ -19,6 +19,6 @@
     <joint name="mobile_base_Revolute_2">
       <command_interface name="effort">
-        <param name="min">-5</param>
-        <param name="max">5</param>
+        <param name="min">-10</param>
+        <param name="max">10</param>
       </command_interface>
       <state_interface name="position"/>
@@ -29,6 +29,16 @@
     <joint name="mobile_base_Revolute_3">
       <command_interface name="effort">
-        <param name="min">-5</param>
-        <param name="max">5</param>
+        <param name="min">-10</param>
+        <param name="max">10</param>
+      </command_interface>
+      <state_interface name="position"/>
+      <state_interface name="velocity"/>
+      <state_interface name="effort"/>
+    </joint>
+    <!-- Joint 4 -->
+    <joint name="mobile_base_Revolute_4">
+       <command_interface name="effort">
+        <param name="min">-10</param>
+        <param name="max">10</param>
       </command_interface>
       <state_interface name="position"/>
@@ -37,7 +47,4 @@
     </joint>
   </ros2_control>
-  <!-- Gazebo ros2_control plugin -->
-  <!-- src/mobile_robot/config/my_controller.yaml -->
-  <!-- $(find mobile_robot)/config/my_controller.yaml -->
   <gazebo>
     <plugin name="gazebo_ros2_control" filename="libgazebo_ros2_control.so">

Commit message: have made the 3d camera sensor and the movable manipulator

File: src/mobile_robot/urdf/robot.urdf.xacro (robot description, xacro)
@@ -1,7 +1,18 @@
 <?xml version="1.0"?>
 <robot xmlns:xacro="http://www.ros.org/wiki/xacro" name="mobile_robot">
-  <!-- shitty file for our robot -->
   <xacro:include filename="robot.xacro"/>
   <xacro:include filename="ros2_control.xacro"/>
-  <!-- <xacro:include filename="lidar.xacro"/> -->
+  <xacro:include filename="$(find ur_description)/urdf/ur_macro.xacro"/>
+  <xacro:include filename="Realsense.xacro"/>
+  <xacro:ur_robot
+    name="ur5"
+    tf_prefix="ur5_"
+    parent="base_link"
+    joint_limits_parameters_file="$(find ur_description)/config/ur5/joint_limits.yaml"
+    kinematics_parameters_file="$(find ur_description)/config/ur5/default_kinematics.yaml"
+    physical_parameters_file="$(find ur_description)/config/ur5/physical_parameters.yaml"
+    visual_parameters_file="$(find ur_description)/config/ur5/visual_parameters.yaml">
+    <origin xyz="0.35 0.0 0.20" rpy="0 0 0" />
+    <xacro:property name="initial_positions" value="${dict(shoulder_pan_joint=1.57, shoulder_lift_joint=-1.57, elbow_joint=0.0, wrist_1_joint=-1.57, wrist_2_joint=0.0, wrist_3_joint=0.0)}" />
+  </xacro:ur_robot>
 </robot>

File: src/mobile_robot/urdf/robot.xacro (robot description, xacro)
@@ -110,5 +110,5 @@
   </link>
   <joint name="camera_joint" type="fixed">
-    <origin xyz="0.474 0.0 0.1355" rpy="-3.14159 -1.57079 0"/>
+    <origin xyz="0.474 0.0 0.1355" rpy="0 0 0"/>
     <parent link="base_link"/><child link="realsense"/>
   </joint>
@@ -124,5 +124,5 @@
   </gazebo>
   <gazebo reference="omni_wheel_1">
-    <mu1>1.5</mu1>
+    <mu1>2.0</mu1>
     <mu2>0.01</mu2>
     <fdir1>1 0 0</fdir1>
@@ -131,5 +131,5 @@
   </gazebo>
   <gazebo reference="omni_wheel_2">
-    <mu1>1.5</mu1>
+    <mu1>2.0</mu1>
     <mu2>0.01</mu2>
     <fdir1>1 0 0</fdir1>
@@ -138,5 +138,5 @@
   </gazebo>
   <gazebo reference="omni_wheel_3">
-    <mu1>1.5</mu1>
+    <mu1>2.0</mu1>
     <mu2>0.01</mu2>
     <fdir1>1 0 0</fdir1>
@@ -145,5 +145,5 @@
   </gazebo>
   <gazebo reference="omni_wheel_4">
-    <mu1>1.5</mu1>
+    <mu1>2.0</mu1>
     <mu2>0.01</mu2>
     <fdir1>1 0 0</fdir1>

File: src/mobile_robot/urdf/ros2_control.xacro (robot description, xacro)
@@ -9,8 +9,14 @@
     <joint name="mobile_base_Revolute_3"><command_interface name="effort"><param name="min">-10</param><param name="max">10</param></command_interface><state_interface name="position"/><state_interface name="velocity"/></joint>
     <joint name="mobile_base_Revolute_4"><command_interface name="effort"><param name="min">-10</param><param name="max">10</param></command_interface><state_interface name="position"/><state_interface name="velocity"/></joint>
+    <joint name="ur5_shoulder_pan_joint"><command_interface name="position"/><state_interface name="position"/><state_interface name="velocity"/></joint>
+    <joint name="ur5_shoulder_lift_joint"><command_interface name="position"/><state_interface name="position"/><state_interface name="velocity"/></joint>
+    <joint name="ur5_elbow_joint"><command_interface name="position"/><state_interface name="position"/><state_interface name="velocity"/></joint>
+    <joint name="ur5_wrist_1_joint"><command_interface name="position"/><state_interface name="position"/><state_interface name="velocity"/></joint>
+    <joint name="ur5_wrist_2_joint"><command_interface name="position"/><state_interface name="position"/><state_interface name="velocity"/></joint>
+    <joint name="ur5_wrist_3_joint"><command_interface name="position"/><state_interface name="position"/><state_interface name="velocity"/></joint>
   </ros2_control>
   <gazebo>
     <plugin filename="libgz_ros2_control-system.so" name="gz_ros2_control::GazeboSimROS2ControlPlugin">
-      <parameters>$(find mobile_robot)/config/my_controller.yaml</parameters>
+      <parameters>$(find mobile_robot)/config/mobile_controller.yaml</parameters>
     </plugin>
   </gazebo>
